Commit message: 1. Self design kobuki_description, add wall distance sensor (following wall behavior) and ultrasonic sensor in the urdf file, so tf transform will publish their transformations
2. add hokuyo laser sensor in the gazebo simulation with kobuki

3. kobuki_driver add more sound playing options in the code, so it can play more than six sounds

4. kobuki_node add ultrasonic and wall distance sensor data publisher in the kobuki_ros, so there are extra two /mobile_base/sensors/* topics to publish sensor data

change subscriber_callback to adopt to play more than six sounds

5. change safety controller behavior. Center bumper activated will move backward certain distance and rotate certain angle based on time. Same for left and right bumper. We can change parameters to control its backward distance and rotation angle

File: kobuki_description/urdf/kobuki_gazebo.urdf.xacro (robot description, xacro)
@@ -42,5 +42,5 @@
 	      <visualize>true</visualize>
 	      <contact>
-	        <collision>base_footprint_fixed_joint_lump__base_collision</collision>
+	        <collision>base_footprint_collision_base_link</collision>
 	      </contact>
 	    </sensor>
